File: bipolar_current_control/bipolar_current_control.kicad_pcb (KiCad board)
At the start: 4 copper layers, 100 x 100 mm, 31 parts, among them J1 Conn_01x10_Pin, J10 Output, J11 Conn_Coaxial, J2 Conn_01x10_Pin, J4 Conn_01x05, J6 Setpoint, J7 Monitor, J8 Current in +, J9 Current in -, Q1 TIP41C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

Commit message: update circuit with op amp power selection
Parts:
- added J3: Conn_01x03_Pin, Connector_PinHeader_2.54mm:PinHeader_1x03_P2.54mm_Vertical, F.Cu at (161.7, 76.2)
- added J5: Conn_01x03_Pin, Connector_PinHeader_2.54mm:PinHeader_1x03_P2.54mm_Vertical, F.Cu at (161.7, 71.1)
- added R9 (alternative footprint for shunt resistor): 2.5R, Resistor_THT:R_Axial_Power_L25.0mm_W9.0mm_P30.48mm, F.Cu at (169.6, 129.5)
- D1, D2: value 3.6V -> 2.5V
- R1: value 2.5R -> 2R; footprint Resistor_THT:R_Axial_Power_L25.0mm_W9.0mm_P30.48mm -> Package_TO_SOT_THT:TO-220F-2_Horizontal_TabUp
- R6: value 100R -> 47R
- moved R1 7.11 mm to (163.1, 127.0), turned to -90 degrees
Connections:
- net Net-(J8-In) renamed /V+
- net Net-(J9-In) renamed /V-
- C1 pad 1: +12V -> /Vs+
- C2 pad 1: +12V -> /Vs+
- C3 pad 1: -12V -> /Vs-
- C4 pad 1: -12V -> /Vs-
- U1 pad 4: -12V -> /Vs-
- U1 pad 8: +12V -> /Vs+
Routing:
- net /V-: track 32.6 -> 81.9 mm
- net /V+: track 32.6 -> 76.8 mm
- net /Vs-: track 0.00 -> 32.6 mm
- net -12V: track 121.7 -> 91.0 mm
- net GND: track 89.8 -> 67.7 mm
- net /Vs+: track 0.00 -> 11.5 mm
- net +12V: track 90.4 -> 80.4 mm
- net /measure: track 72.8 -> 75.4 mm
Other:
- board text added: "Op amp power select +-12V / Current-supply"

Commit message: add design with ADA4700-1
Changed lines of the file:
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@@
 		(property "Value" "AD823"
 			(at 3.81 9.95 0)
-			(layer "F.Fab")
+			(layer "F.SilkS")
 			(effects
 				(font
