File: bipolar_current_driver_ADA4700-1/bipolar_current_driver_ADA4700-1.kicad_pcb (KiCad board)
At the start: 4 copper layers, 100 x 100 mm, 40 parts, among them J1 Conn_01x10_Pin, J10 Output, J11 Conn_Coaxial, J2 Conn_01x10_Pin, J4 Conn_01x05, J5 Screw_Terminal_01x02, J6 Setpoint, J7 Conn_Coaxial, J8 V+, J9 V-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

Commit message: add production files
Parts:
- J5: value Screw_Terminal_01x02 -> +12 V for fans
Changed lines of the file:
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@@
 			(drillshape 0)
 			(scaleselection 1)
-			(outputdirectory "./production/")
+			(outputdirectory "production/gerber/")
 		)
 	)
@@
 		)
 		(property "Value" "TIP42C"
-			(at 2.54 -2 0)
-			(layer "F.Fab")
+			(at 2.54 9.23 0)
+			(layer "F.SilkS")
 			(effects
 				(font
@@
 		)
 		(property "Value" "2R"
-			(at 2.54 -2 0)
-			(layer "F.Fab")
+			(at 2.54 9.23 0)
+			(layer "F.SilkS")
 			(effects
 				(font
@@
 		)
 		(property "Value" "LM317HV"
-			(at 2.54 -2 0)
-			(layer "F.Fab")
+			(at 2.54 9.23 0)
+			(layer "F.SilkS")
 			(effects
 				(font
@@
 		)
 		(property "Value" "TIP41C"
-			(at 2.54 -2 0)
-			(layer "F.Fab")
+			(at 2.54 9.23 0)
+			(layer "F.SilkS")
 			(effects
 				(font
@@
 			)
 		)
-		(property "Value" "Screw_Terminal_01x02"
+		(property "Value" "+12 V for fans"
 			(at 2.78 7.75 0)
-			(layer "F.Fab")
+			(layer "F.SilkS")
 			(effects
 				(font
