File: bipolar_current_driver_ADA4700-1/bipolar_current_driver_ADA4700-1.kicad_sch (KiCad schematic)
At the start: 37 parts, among them J1 Conn_01x10_Pin, J10 Output, J11 Conn_Coaxial, J2 Conn_01x10_Pin, J4 Conn_01x05, J5 Screw_Terminal_01x02, J6 Setpoint, J7 Conn_Coaxial, J8 V+, J9 V-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

Commit message: add production files
Other:
- company: (none) -> UC Berkeley
- title: ??? -> Bipolar Current Driver
Changed lines of the file:
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@@
 	(paper "A4")
 	(title_block
-		(title "???")
-		(comment 1 "Designed by Jack Roth")
-		(comment 2 "Compatible with Hammond Manufacturing series 1457")
+		(title "Bipolar Current Driver")
+		(company "UC Berkeley")
+		(comment 1 "Y. Yang")
 	)
 	(text "Solder wire connections"
